File: AE101Corolla.kicad_pcb (KiCad board)
At the start: 4 copper layers, 100 x 100 mm, 13 parts, among them J1 175448-6, M1 Module-mega-mcu144-0.7, M2 Module-vr-discrete-0.5, M3 Module-vr-max9924-0.1, M4 Module-power_12and5V-0.3

Commit message: sync
Parts:
- added J2: 6437288-2, 6437288_2:TE_6437288-2, F.Cu at (118.8, 124.8)
- added J3: USB_C_Receptacle_USB2.0_14P, Connector_USB:USB_C_Receptacle_GCT_USB4105-xx-A_16P_TopMnt_Horizontal, F.Cu at (144.2, 147.0)
- added JP1: SolderJumper_2_Open, Jumper:SolderJumper-2_P1.3mm_Open_TrianglePad1.0x1.5mm, F.Cu at (30.9, 129.8)
- added M5: Module-knock-0.2, knock:knock, F.Cu at (143.0, 68.7)
- added M6: Module-can-0.1, can:can, F.Cu at (121.9, 100.7)
- added R1: 4.7k, Resistor_SMD:R_0402_1005Metric, F.Cu at (27.2, 129.0)
- added R2: 4.7k, Resistor_SMD:R_0402_1005Metric, F.Cu at (27.2, 131.0)
- added R3: 4.7k, Resistor_SMD:R_0402_1005Metric, F.Cu at (27.2, 133.0)
- added R4: 4.7k, Resistor_SMD:R_0402_1005Metric, F.Cu at (27.2, 135.0)
- added R5: 5.1k, Resistor_SMD:R_0402_1005Metric, F.Cu at (68.0, 102.1)
- added R6: 5.1k, Resistor_SMD:R_0402_1005Metric, F.Cu at (68.0, 104.1)
- M1: footprint megamcu144:mega-mcu144 -> mega-mcu144:mega-mcu144
- M3: footprint vrmax9924:vr-max9924 -> vr-max9924:vr-max9924
- M4: footprint power5_12:power_12and5V -> power_12and5V:power_12and5V
- moved D2 157.7 mm to (35.8, 146.2)
- moved D3 157.7 mm to (35.8, 149.5)
- moved D4 157.7 mm to (35.8, 152.9)
- moved D1 157.7 mm to (35.8, 142.8)
- moved U3 133.4 mm to (50.8, 105.6)
- moved U4 133.4 mm to (50.8, 112.2), turned to 180 degrees
- moved U1 132.9 mm to (50.8, 92.5)
- moved U2 132.9 mm to (50.8, 99.1)
- moved M3 66.2 mm to (159.7, 68.3), turned to -90 degrees
- moved M2 58.2 mm to (169.7, 68.3), turned to -90 degrees
- moved M1 53.7 mm to (182.0, 97.3), turned to 180 degrees
- moved M4 44.3 mm to (119.4, 90.5)
- moved J1 0.25 mm to (194.1, 63.8)
Connections:
- D2 pad 2: Net-(D2-A) -> /BOOSTSOLENOID_OUT
- D3 pad 2: /IATOPEN_OUT -> /IACOPEN_OUT
- D4 pad 2: /IATCLOSE_OUT -> /IACCLOSE_OUT
- J1 pad 1: unconnected-(J1-Pad1) -> GND
- J1 pad 11: unconnected-(J1-ACT-Pad11) -> /ACTEMP
- J1 pad 13: unconnected-(J1-FC-Pad13) -> /FUELRELAY_OUT
- J1 pad 15: unconnected-(J1-BATT-Pad15) -> +12V_PERM
- J1 pad 16: unconnected-(J1-+B1-Pad16) -> +12V_RAW
- J1 pad 17: unconnected-(J1-ELS-Pad17) -> /ELECTRICLOAD
- J1 pad 18: unconnected-(J1-SPD-Pad18) -> /SPEED
- J1 pad 19: unconnected-(J1-AC1-Pad19) -> /ACSTATUS
- J1 pad 2: unconnected-(J1-Pad2) -> /INJ1_OUT
- J1 pad 21: unconnected-(J1-W?-Pad21) -> /CHECKENGINE
- J1 pad 22: unconnected-(J1-+B-Pad22) -> +12V_RAW
- J1 pad 23: unconnected-(J1-Pad23) -> /IACOPEN_OUT
- J1 pad 24: unconnected-(J1-Pad24) -> /IACCLOSE_OUT
- J1 pad 28: unconnected-(J1-Pad28) -> /SYNC+
- J1 pad 29: unconnected-(J1-Pad29) -> /VR+
- J1 pad 32: unconnected-(J1-Pad32) -> /IGN1
- J1 pad 36: unconnected-(J1-Pad36) -> /SYNC-
- J1 pad 37: unconnected-(J1-Pad37) -> /VR-
- J1 pad 41: unconnected-(J1-Pad41) -> /NARROWO2_UPSTR
- J1 pad 42: unconnected-(J1-Pad42) -> /NARROWO2_DOWNSTR
- J1 pad 43: unconnected-(J1-Pad43) -> /CLT
- J1 pad 44: unconnected-(J1-Pad44) -> /IAT
- J1 pad 45: unconnected-(J1-Pad45) -> /MAP
- J1 pad 47: unconnected-(J1-Pad47) -> GND
- J1 pad 49: unconnected-(J1-Pad49) -> /KNOCK_RAW
- J1 pad 51: unconnected-(J1-Pad51) -> /IDLSW
- J1 pad 52: unconnected-(J1-Pad52) -> +5VP
- J1 pad 53: unconnected-(J1-Pad53) -> /TPS
- J1 pad 54: unconnected-(J1-Pad54) -> GNDA
- J1 pad 6: unconnected-(J1-Pad6) -> GND
- J1 pad 7: unconnected-(J1-Pad7) -> /INJ3_OUT
- J1 pad 8: unconnected-(J1-Pad8) -> GND
- J1 pad 9: unconnected-(J1-Pad9) -> /NEUTRALSW
- M1 pad E1: unconnected-(M1-SPI2_SCK/CAN2_TX-PadE1) -> Net-(M1-SPI2_SCK/CAN2_TX)
- M1 pad E16: unconnected-(M1-OUT_PWM3-PadE16) -> /BOOSTSOLENOID_IN
- M1 pad E17: unconnected-(M1-OUT_PWM2-PadE17) -> /IACOPEN_IN
- M1 pad E27: unconnected-(M1-OUT_PWM1-PadE27) -> /IACCLOSE_IN
- M1 pad E28: unconnected-(M1-OUT_PWM8-PadE28) -> /VR_THRESH
- M1 pad E31: unconnected-(M1-OUT_INJ5-PadE31) -> /FUELRELAY_IN
- M1 pad E38: unconnected-(M1-V5A_SWITCHABLE-PadE38) -> +5VA
- M1 pad E4: unconnected-(M1-SPI2_CS/CAN2_RX-PadE4) -> Net-(M1-SPI2_CS/CAN2_RX)
- M1 pad N2: unconnected-(M1-USBM-PadN2) -> /USB-
- M1 pad N26: unconnected-(M1-IN_VIGN-PadN26) -> /VIGN
- M1 pad N27: unconnected-(M1-VBAT-PadN27) -> /VBAT
- M1 pad N28: unconnected-(M1-V33_SWITCHABLE-PadN28) -> +3.3VA
- M1 pad N29: unconnected-(M1-OUT_PWR_EN-PadN29) -> /5VP_ENABLE
- M1 pad N3: unconnected-(M1-USBP-PadN3) -> /USB+
- M1 pad N31: unconnected-(M1-VCC-PadN31) -> +5V
- M1 pad N4: unconnected-(M1-VBUS-PadN4) -> Net-(M1-VBUS)
- M1 pad S1: unconnected-(M1-IN_D4-PadS1) -> /IDLSW
- M1 pad S10: unconnected-(M1-IN_AUX4-PadS10) -> /AUX4
- M1 pad S11: unconnected-(M1-IN_AUX3-PadS11) -> /AUX3
- M1 pad S12: unconnected-(M1-IN_AUX2-PadS12) -> /AUX2
- M1 pad S13: unconnected-(M1-IN_AUX1-PadS13) -> /AUX1
- M1 pad S14: unconnected-(M1-IN_RES2-PadS14) -> /RES2
- M1 pad S15: unconnected-(M1-IN_O2S2-PadS15) -> /NARROWO2_DOWNSTR
- M1 pad S16: unconnected-(M1-IN_O2S-PadS16) -> /NARROWO2_UPSTR
- M1 pad S17: unconnected-(M1-IN_RES1-PadS17) -> /RES1
- M1 pad S18: unconnected-(M1-IN_RES3-PadS18) -> /RES3
- M1 pad S2: unconnected-(M1-IN_D3-PadS2) -> /ACSTATUS
- M1 pad S21: unconnected-(M1-IN_MAP1-PadS21) -> /MAP
- M1 pad S22: unconnected-(M1-IN_CRANK-PadS22) -> /MAINVR_OUT
- M1 pad S23: unconnected-(M1-IN_KNOCK-PadS23) -> /KNOCK_PROCESSED
- M1 pad S24: unconnected-(M1-IN_CAM-PadS24) -> /SYNCVR_OUT
- M1 pad S25: unconnected-(M1-IN_VSS-PadS25) -> /SPEED
- M1 pad S26: unconnected-(M1-IN_IAT-PadS26) -> /IAT
- M1 pad S28: unconnected-(M1-IN_CLT-PadS28) -> /CLT
- M1 pad S3: unconnected-(M1-IN_D2-PadS3) -> /ELECTRICLOAD
- M1 pad S30: unconnected-(M1-IN_TPS-PadS30) -> /TPS
- M1 pad S35: unconnected-(M1-VREF1-PadS35) -> /VREF1
- M1 pad W1: unconnected-(M1-GNDA-PadW1) -> GNDA
- M1 pad W10: unconnected-(M1-IGN2-PadW10) -> /IGN2
- M1 pad W11: unconnected-(M1-IGN1-PadW11) -> /IGN1
- M1 pad W12: unconnected-(M1-CANH-PadW12) -> /CAN1H
- M1 pad W13: unconnected-(M1-CANL-PadW13) -> /CAN1L
- M1 pad W8: unconnected-(M1-IGN4-PadW8) -> /IGN4
- M1 pad W9: unconnected-(M1-IGN3-PadW9) -> /IGN3
- M2 pad E1: unconnected-(M2-Thresh_IN-PadE1) -> /VR_THRESH
- M2 pad E3: unconnected-(M2-OUT-PadE3) -> /SYNCVR_OUT
- M2 pad E4: unconnected-(M2-V5_IN-PadE4) -> +5VA
- M2 pad G: unconnected-(M2-GND-PadG) -> GND
- M2 pad W1: unconnected-(M2-VR--PadW1) -> /SYNC-
- M2 pad W2: unconnected-(M2-VR+-PadW2) -> /SYNC+
- M3 pad E1: unconnected-(M3-HALL_EN-PadE1) -> Net-(JP1-A)
- M3 pad E3: unconnected-(M3-OUT-PadE3) -> /MAINVR_OUT
- M3 pad E4: unconnected-(M3-V5_IN-PadE4) -> +5VA
- M3 pad G: unconnected-(M3-GND-PadG) -> GND
- M3 pad W1: unconnected-(M3-VR-/HALL-PadW1) -> /VR-
- M3 pad W2: unconnected-(M3-VR+-PadW2) -> /VR+
- M4 pad E1: unconnected-(M4-VBAT-PadE1) -> /VBAT
- M4 pad E3: unconnected-(M4-VIGN-PadE3) -> /VIGN
- M4 pad E4: unconnected-(M4-V5-PadE4) -> +5V
- M4 pad E5: unconnected-(M4-EN_5VP-PadE5) -> /5VP_ENABLE
- M4 pad S1: unconnected-(M4-GND-PadS1) -> GND
- M4 pad V1: unconnected-(M4-V12_PERM-PadV1) -> +12V_PERM
- M4 pad V2: unconnected-(M4-IN_VIGN-PadV2) -> +12V_RAW
- M4 pad V3: unconnected-(M4-V12_RAW-PadV3) -> +12V_RAW
- M4 pad V4: unconnected-(M4-5VP-PadV4) -> +5VP
- U3 pad 1: unconnected-(U3-IN1-Pad1) -> /BOOSTSOLENOID_IN
- U3 pad 5: /FUELRELAY_OUT -> GND
- U3 pad 6: unconnected-(U3-DRAIN2-Pad6) -> /FUELRELAY_OUT
- U3 pad 7: Net-(D2-A) -> GND
- U3 pad 8: unconnected-(U3-DRAIN1-Pad8) -> /BOOSTSOLENOID_OUT
- U4 pad 1: /IATCLOSE_IN -> /IACCLOSE_IN
- U4 pad 3: /IATOPEN_IN -> /IACOPEN_IN
- U4 pad 5: /IATOPEN_OUT -> GND
- U4 pad 6: unconnected-(U4-DRAIN2-Pad6) -> /IACOPEN_OUT
- U4 pad 7: /IATCLOSE_OUT -> GND
- U4 pad 8: unconnected-(U4-DRAIN1-Pad8) -> /IACCLOSE_OUT
Routing:
- net /VR-: track 0.00 -> 12.3 mm
- net /SYNC-: track 0.00 -> 10.6 mm
- net /KNOCK_RAW: track 0.00 -> 10.3 mm
- net /VR+: track 0.00 -> 6.51 mm
- net /SYNC+: track 0.00 -> 5.71 mm
- net +12V_RAW: track 0.00 -> 4.50 mm

Commit message: sync
Parts:
- added D5: B5819W, Diode_SMD:D_SOD-123, B.Cu at (195.5, 131.0)
- added D6: B5819W, Diode_SMD:D_SOD-123, B.Cu at (190.5, 131.0)
- added D7: B5819W, Diode_SMD:D_SOD-123, B.Cu at (198.0, 131.0)
- added D8: B5819W, Diode_SMD:D_SOD-123, B.Cu at (193.0, 131.0)
- added R10: 4.7k, Resistor_SMD:R_0402_1005Metric, F.Cu at (227.8, 90.0)
- added R7: 4.7k, Resistor_SMD:R_0402_1005Metric, F.Cu at (227.8, 84.0)
- added R8: 4.7k, Resistor_SMD:R_0402_1005Metric, F.Cu at (227.8, 86.0)
- added R9: 4.7k, Resistor_SMD:R_0402_1005Metric, F.Cu at (227.8, 88.0)
- added U5: ~, VNLD5090-E:VNLD5090-E, B.Cu at (193.8, 118.8)
- added U6: ~, VNLD5090-E:VNLD5090-E, B.Cu at (193.8, 125.0)
- D1, D2, D3, D4, U1, U2: moved to B.Cu
- moved D3 170.0 mm to (184.5, 67.0), turned to 90 degrees
- moved D4 168.9 mm to (181.2, 67.0), turned to 90 degrees
- moved U1 143.6 mm to (193.8, 105.5), turned to 180 degrees
- moved U2 143.5 mm to (193.8, 111.5), turned to 180 degrees
- moved U4 138.7 mm to (183.5, 71.8), turned to 90 degrees
- moved M6 134.3 mm to (247.6, 148.1)
- moved D2 109.5 mm to (112.0, 67.5), turned to 90 degrees
- moved D1 109.4 mm to (115.2, 67.5), turned to 90 degrees
- moved J3 101.7 mm to (242.1, 119.4)
- moved U3 71.9 mm to (114.2, 71.8), turned to 90 degrees
- moved JP1 70.7 mm to (83.5, 82.5)
- moved J2 66.0 mm to (184.2, 116.8), turned to 90 degrees
- moved M4 53.5 mm to (106.9, 142.5)
- moved M1 50.7 mm to (166.4, 145.5), turned to 90 degrees
- moved M3 0.50 mm to (159.2, 68.3)
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Connections:
- D2 pad 2: /BOOSTSOLENOID_OUT -> /CHECKENGINE_OUT
- J1 pad 21: /CHECKENGINE -> /CHECKENGINE_OUT
- J1 pad 47: GND -> GNDA
- J2 pad 1: /INJ1_OUT -> unconnected-(J2-Pad1)
- J2 pad 10: /AUX1 -> unconnected-(J2-Pad10)
- J2 pad 11: /AUX2 -> unconnected-(J2-Pad11)
- J2 pad 12: /AUX3 -> unconnected-(J2-Pad12)
- J2 pad 13: /AUX4 -> unconnected-(J2-Pad13)
- J2 pad 2: /INJ2_OUT -> unconnected-(J2-Pad2)
- J2 pad 26: /RES1 -> unconnected-(J2-Pad26)
- J2 pad 27: /RES2 -> /LS4_OUT
- J2 pad 28: /RES3 -> /LS3_OUT
- J2 pad 29: unconnected-(J2-Pad29) -> /LS2_OUT
- J2 pad 3: /INJ3_OUT -> unconnected-(J2-Pad3)
- J2 pad 30: unconnected-(J2-Pad30) -> /LS1_OUT
- J2 pad 31: unconnected-(J2-Pad31) -> /INJ4_OUT
- J2 pad 32: unconnected-(J2-Pad32) -> /INJ3_OUT
- J2 pad 33: unconnected-(J2-Pad33) -> /INJ2_OUT
- J2 pad 34: unconnected-(J2-Pad34) -> /INJ1_OUT
- J2 pad 4: /INJ4_OUT -> unconnected-(J2-Pad4)
- J2 pad 5: /BOOSTSOLENOID_OUT -> unconnected-(J2-Pad5)
- J2 pad 6: /IGN1 -> unconnected-(J2-Pad6)
- J2 pad 7: /IGN2 -> unconnected-(J2-Pad7)
- J2 pad 8: /IGN3 -> unconnected-(J2-Pad8)
- J2 pad 9: /IGN4 -> unconnected-(J2-Pad9)
- JP1 pad 2: +5V -> +5VA
- M1 pad E14: unconnected-(M1-OUT_PWM5-PadE14) -> /LS3_IN
- M1 pad E15: unconnected-(M1-OUT_PWM4-PadE15) -> /LS2_IN
- M1 pad E16: /BOOSTSOLENOID_IN -> /LS1_IN
- M1 pad E17: /IACOPEN_IN -> /LS4_IN
- M1 pad E18: /INJ2_IN -> /CHECKENGINE_IN
- M1 pad E19: /INJ1_IN -> /FUELRELAY_IN
- M1 pad E26: unconnected-(M1-OUT_PWM6-PadE26) -> /IACOPEN_IN
- M1 pad E29: /INJ3_IN -> unconnected-(M1-OUT_INJ3-PadE29)
- M1 pad E30: /INJ4_IN -> unconnected-(M1-OUT_INJ4-PadE30)
- M1 pad E31: /FUELRELAY_IN -> /INJ4_IN
- M1 pad E32: unconnected-(M1-OUT_INJ6-PadE32) -> /INJ3_IN
- M1 pad E33: unconnected-(M1-OUT_INJ7-PadE33) -> /INJ2_IN
- M1 pad E34: unconnected-(M1-OUT_INJ8-PadE34) -> /INJ1_IN
- M1 pad S19: unconnected-(M1-IN_MAP3-PadS19) -> /ACSTATUS
- M1 pad S2: /ACSTATUS -> /D3
- M1 pad S20: unconnected-(M1-IN_MAP2-PadS20) -> /ELECTRICLOAD
- M1 pad S3: /ELECTRICLOAD -> /D2
- M1 pad S4: unconnected-(M1-IN_D1-PadS4) -> /D1
- M1 pad S6: unconnected-(M1-IN_SENS4-PadS6) -> /SENS4
- M1 pad S7: unconnected-(M1-IN_SENS3-PadS7) -> /SENS3
- M1 pad S8: unconnected-(M1-IN_SENS2-PadS8) -> /SENS2
- M1 pad S9: unconnected-(M1-IN_SENS1-PadS9) -> /SENS1
- R3 pad 1: /BOOSTSOLENOID_IN -> /CHECKENGINE_IN
- U1 pad 6: Net-(U1-DRAIN1) -> GND
- U1 pad 8: Net-(U1-DRAIN1) -> GND
- U3 pad 1: /BOOSTSOLENOID_IN -> /CHECKENGINE_IN
- U3 pad 8: /BOOSTSOLENOID_OUT -> /CHECKENGINE_OUT
Routing:
- net +5VP: track 0.00 -> 119.5 mm
- net /LS4_IN: track 0.00 -> 95.8 mm, vias 0 -> 3
- net /LS3_IN: track 0.00 -> 93.8 mm, vias 0 -> 3
- net /LS2_IN: track 0.00 -> 89.7 mm, vias 0 -> 3
- net /LS1_IN: track 0.00 -> 83.6 mm, vias 0 -> 3
- net +12V_RAW: track 4.50 -> 76.8 mm
- net /IACOPEN_IN: track 0.00 -> 61.4 mm, vias 0 -> 2
- net /INJ4_IN: track 0.00 -> 60.2 mm, vias 0 -> 2
- net +12V_PERM: track 0.00 -> 59.5 mm
- net /IACCLOSE_IN: track 0.00 -> 59.0 mm, vias 0 -> 2
- net /INJ3_OUT: track 0.00 -> 58.9 mm
- net /INJ3_IN: track 0.00 -> 55.0 mm, vias 0 -> 2
- net /SYNCVR_OUT: track 0.00 -> 53.2 mm
- net /INJ2_IN: track 0.00 -> 50.1 mm, vias 0 -> 2
- net /MAINVR_OUT: track 0.00 -> 46.6 mm
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
Commit message: sync
Parts:
- added M7: Module-wbo-0.5, wbo:wbo, F.Cu at (211.8, 106.4)
- D5, D6, D7, D8: moved to F.Cu
- J2: footprint 6437288_2:TE_6437288-2 -> superseal_34:TE_6437288-2
- M1: footprint mega-mcu144:mega-mcu144 -> megamcu144:mega-mcu144
- M3: footprint vr-max9924:vr-max9924 -> vrmax9924:vr-max9924
- M4: footprint power_12and5V:power_12and5V -> power5_12:power_12and5V
- R1, R2, R5, R6: moved to B.Cu
- moved R2 186.0 mm to (199.5, 61.0), turned to 90 degrees
- moved R1 182.7 mm to (196.8, 61.0), turned to 90 degrees
- moved R4 120.7 mm to (140.8, 94.0), turned to -90 degrees
- moved R3 117.9 mm to (138.5, 94.0), turned to -90 degrees
- moved J3 93.8 mm to (149.8, 135.8)
- moved R7 90.9 mm to (140.0, 107.8), turned to -90 degrees
- moved JP1 89.9 mm to (172.3, 68.8), turned to 180 degrees
- moved R9 88.7 mm to (141.2, 107.8), turned to -90 degrees
- moved R5 88.7 mm to (150.5, 134.8), turned to 90 degrees
- moved R8 88.0 mm to (142.5, 107.8), turned to -90 degrees
- moved R6 87.1 mm to (149.5, 134.8), turned to 90 degrees
- moved R10 85.9 mm to (143.8, 107.8), turned to -90 degrees
- moved U6 79.6 mm to (121.2, 92.1), turned to 0 degrees
- moved U2 78.9 mm to (121.2, 80.2), turned to 0 degrees
- moved U5 75.3 mm to (121.2, 98.2), turned to 0 degrees
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Connections:
- J1 pad 2: /INJ1_OUT -> unconnected-(J1-#10-Pad2)
- J1 pad 7: /INJ3_OUT -> unconnected-(J1-#20-Pad7)
- J2 pad 1: unconnected-(J2-Pad1) -> /IGN1
- J2 pad 10: unconnected-(J2-Pad10) -> /AUX1
- J2 pad 11: unconnected-(J2-Pad11) -> /AUX2
- J2 pad 12: unconnected-(J2-Pad12) -> /AUX3
- J2 pad 13: unconnected-(J2-Pad13) -> /AUX4
- J2 pad 18: unconnected-(J2-Pad18) -> /RES1
- J2 pad 19: unconnected-(J2-Pad19) -> /RES3
- J2 pad 2: unconnected-(J2-Pad2) -> /IGN2
- J2 pad 20: unconnected-(J2-Pad20) -> /RES2
- J2 pad 21: unconnected-(J2-Pad21) -> /D2
- J2 pad 22: unconnected-(J2-Pad22) -> /OUT1
- J2 pad 23: unconnected-(J2-Pad23) -> /OUT2
- J2 pad 24: unconnected-(J2-Pad24) -> /OUT3
- J2 pad 25: unconnected-(J2-Pad25) -> /OUT4
- J2 pad 26: unconnected-(J2-Pad26) -> /D3
- J2 pad 27: /LS4_OUT -> /INJ4_OUT
- J2 pad 28: /LS3_OUT -> /INJ3_OUT
- J2 pad 29: /LS2_OUT -> /INJ2_OUT
- J2 pad 3: unconnected-(J2-Pad3) -> /IGN3
- J2 pad 30: /LS1_OUT -> /INJ1_OUT
- J2 pad 31: /INJ4_OUT -> /LS4_OUT
- J2 pad 32: /INJ3_OUT -> /LS3_OUT
- J2 pad 33: /INJ2_OUT -> /LS2_OUT
- J2 pad 34: /INJ1_OUT -> /LS1_OUT
- J2 pad 4: unconnected-(J2-Pad4) -> /IGN4
- J2 pad 5: unconnected-(J2-Pad5) -> /SENS1
- J2 pad 6: unconnected-(J2-Pad6) -> /SENS2
- J2 pad 7: unconnected-(J2-Pad7) -> /SENS3
- J2 pad 8: unconnected-(J2-Pad8) -> /SENS4
- J2 pad 9: unconnected-(J2-Pad9) -> /D1
- M1 pad E14: /LS3_IN -> /LS4_IN
- M1 pad E15: /LS2_IN -> /LS3_IN
- M1 pad E16: /LS1_IN -> /LS2_IN
- M1 pad E17: /LS4_IN -> /LS1_IN
- M1 pad E29: unconnected-(M1-OUT_INJ3-PadE29) -> /INJ4_IN
- M1 pad E30: unconnected-(M1-OUT_INJ4-PadE30) -> /INJ3_IN
- M1 pad E31: /INJ4_IN -> /INJ2_IN
- M1 pad E32: /INJ3_IN -> /INJ1_IN
- M1 pad E33: /INJ2_IN -> unconnected-(M1-OUT_INJ7-PadE33)
- M1 pad E34: /INJ1_IN -> unconnected-(M1-OUT_INJ8-PadE34)
- M1 pad E39: unconnected-(M1-GNDA-PadE39) -> GNDA
- M1 pad N30: unconnected-(M1-V5A_SWITCHABLE-PadN30) -> +5VA
- M1 pad S27: unconnected-(M1-IN_AT1-PadS27) -> /ACTEMP
- M1 pad W2: unconnected-(M1-V5A_SWITCHABLE-PadW2) -> +5VA
- M1 pad W4: unconnected-(M1-IGN8-PadW4) -> /OUT4
- M1 pad W5: unconnected-(M1-IGN7-PadW5) -> /OUT3
- M1 pad W6: unconnected-(M1-IGN6-PadW6) -> /OUT2
- M1 pad W7: unconnected-(M1-IGN5-PadW7) -> /OUT1
- U1 pad 5: /INJ2_OUT -> GND
- U1 pad 6: GND -> /INJ2_OUT
- U1 pad 7: /INJ1_OUT -> GND
- U1 pad 8: GND -> /INJ1_OUT
- U2 pad 5: /INJ4_OUT -> GND
- U2 pad 6: GND -> /INJ4_OUT
- U2 pad 7: /INJ3_OUT -> GND
- U2 pad 8: GND -> /INJ3_OUT
Routing:
- net +12V_RAW: track 76.8 -> 190.7 mm, vias 0 -> 3
- net /OUT4: track 0.00 -> 94.8 mm
- net /OUT3: track 0.00 -> 93.5 mm
- net /OUT2: track 0.00 -> 93.2 mm
- net /OUT1: track 0.00 -> 91.8 mm
- net /IGN1: track 0.00 -> 85.9 mm
- net /IGN2: track 0.00 -> 85.8 mm
- net /IGN3: track 0.00 -> 85.1 mm
- net /IGN4: track 0.00 -> 84.8 mm
- net +5VA: track 0.00 -> 59.1 mm, vias 0 -> 1
- net /INJ3_OUT: track 58.9 -> 2.56 mm
- net /SPEED: track 0.00 -> 54.3 mm, vias 0 -> 2
- net /LS3_IN: track 93.8 -> 40.0 mm, vias 3 -> 1
- net /TPS: track 0.00 -> 52.8 mm
- net /LS2_IN: track 89.7 -> 36.9 mm, vias 3 -> 1
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
Commit message: sync
Parts:
- added J4: Conn_02x03_Counter_Clockwise, Connector_Molex:Molex_Mini-Fit_Jr_5569-06A2_2x03_P4.20mm_Horizontal, F.Cu at (206.2, 68.8)
- moved M7 2.58 mm to (210.7, 108.7)
Connections:
- M7 pad E1: unconnected-(M7-LSU_Un-PadE1) -> Net-(J4-Pin_6)
- M7 pad E2: unconnected-(M7-LSU_Vm-PadE2) -> Net-(J4-Pin_4)
- M7 pad E3: unconnected-(M7-LSU_Ip-PadE3) -> Net-(J4-Pin_3)
- M7 pad E4: unconnected-(M7-LSU_Rtrim-PadE4) -> Net-(J4-Pin_1)
- M7 pad E5: unconnected-(M7-LSU_H+-PadE5) -> Net-(J4-Pin_5)
- M7 pad E6: unconnected-(M7-LSU_H--PadE6) -> GND
- M7 pad G: unconnected-(M7-GND-PadG) -> GND
- M7 pad J1: unconnected-(M7-SEL1-PadJ1) -> Net-(M7-PULL_DOWN1)
- M7 pad J_GND1: unconnected-(M7-PULL_DOWN1-PadJ_GND1) -> Net-(M7-PULL_DOWN1)
- M7 pad W1: unconnected-(M7-V5_IN-PadW1) -> +5VA
- M7 pad W2: +3.3VA -> unconnected-(M7-CAN_VIO-PadW2)
Routing:
- net +3.3VA: track 51.1 -> 17.5 mm
- net +12V_RAW: track 190.7 -> 218.1 mm
- net Net-(J4-Pin_4): track 0.00 -> 15.0 mm
- net Net-(J4-Pin_1): track 0.00 -> 13.8 mm
- net Net-(J4-Pin_5): track 0.00 -> 11.1 mm
- net Net-(J4-Pin_6): track 0.00 -> 10.1 mm, vias 0 -> 2
- net Net-(J4-Pin_3): track 0.00 -> 4.71 mm
- net /CAN1L: track 18.2 -> 16.9 mm
- net /CAN1H: track 17.3 -> 16.3 mm

Commit message: sync
Parts:
- added C1: 100n, Capacitor_SMD:C_0402_1005Metric, F.Cu at (204.5, 120.8)
- added C2: 10n, Capacitor_SMD:C_0402_1005Metric, F.Cu at (206.2, 124.0)
- added U7: MAX31855KASA, Package_SO:SOIC-8_3.9x4.9mm_P1.27mm, F.Cu at (202.0, 124.0)
- moved M2 0.50 mm to (185.2, 57.8)
Connections:
- M1 pad E38: +5VA -> unconnected-(M1-V5A_SWITCHABLE-PadE38)
- M1 pad N10: unconnected-(M1-SPI3_CS-PadN10) -> /CS3
- M1 pad N11: unconnected-(M1-SPI3_SCK-PadN11) -> /SCK3
- M1 pad N12: unconnected-(M1-SPI3_MISO-PadN12) -> /MISO3
- M1 pad S35: /VREF1 -> unconnected-(M1-VREF1-PadS35)
- M1 pad S5: unconnected-(M1-VREF2-PadS5) -> /VREF1
- M1 pad W1: GNDA -> unconnected-(M1-GNDA-PadW1)
Routing:
- net GNDA: track 0.00 -> 79.1 mm, vias 0 -> 3
- net +5VA: track 59.1 -> 134.1 mm, vias 1 -> 0
- net /MISO3: track 0.00 -> 48.8 mm, vias 0 -> 1
- net /CS3: track 0.00 -> 48.8 mm
- net /SCK3: track 0.00 -> 48.2 mm
- net /D2: track 0.00 -> 47.5 mm, vias 0 -> 2
- net /D3: track 0.00 -> 35.0 mm, vias 0 -> 2
- net /IGN1: track 85.9 -> 117.7 mm, vias 0 -> 1
- net /NARROWO2_UPSTR: track 0.00 -> 31.4 mm, vias 0 -> 1
- net /VREF1: track 0.00 -> 30.5 mm, vias 0 -> 1
- net /NARROWO2_DOWNSTR: track 0.00 -> 30.3 mm, vias 0 -> 1
- net +5VP: track 123.7 -> 142.4 mm, vias 0 -> 1
- net /VIGN: track 32.0 -> 34.3 mm
- net /EGT-: track 0.00 -> 1.84 mm
- net /EGT+: track 0.00 -> 1.84 mm
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
Commit message: sync
Parts:
- added REF**: MountingHole_3.2mm_M3_Pad_Via, MountingHole:MountingHole_3.2mm_M3_Pad_Via, F.Cu at (119.2, 61.0)
- added REF**: MountingHole_3.2mm_M3_Pad_Via, MountingHole:MountingHole_3.2mm_M3_Pad_Via, F.Cu at (119.2, 136.0)
- added REF**: MountingHole_3.2mm_M3_Pad_Via, MountingHole:MountingHole_3.2mm_M3_Pad_Via, F.Cu at (212.2, 61.0)
- added REF**: MountingHole_3.2mm_M3_Pad_Via, MountingHole:MountingHole_3.2mm_M3_Pad_Via, F.Cu at (212.2, 136.0)
Routing:
- net +12V_RAW: track 218.1 -> 222.4 mm
- net +5VP: track 142.4 -> 146.0 mm
- net +12V_PERM: track 64.1 -> 63.3 mm
- net GND: vias 256 -> 261
