File: AE101Corolla.kicad_pcb (KiCad board)
At the start: 4 copper layers, 100 x 100 mm, 43 parts, among them J1 175448-6, J2 6437288-2, J3 USB_C_Receptacle_USB2.0_14P, J4 Conn_02x03_Counter_Clockwise, M1 Module-mega-mcu144-0.7, M2 Module-vr-discrete-0.5, M3 Module-vr-max9924-0.1, M4 Module-power_12and5V-0.3, M5 Module-knock-0.2, M6 Module-can-0.1, M7 Module-wbo-0.5, U7 MAX31855KASA

Commit message: sync
Parts:
- moved U3 1.34 mm to (130.1, 61.2)
Routing:
- net /CHECKENGINE_IN: track 49.8 -> 48.3 mm
- net /FUELRELAY_OUT: track 9.02 -> 8.47 mm
- net /CHECKENGINE_OUT: track 12.8 -> 13.4 mm
- net /FUELRELAY_IN: track 46.6 -> 46.0 mm
- net GND: vias 261 -> 258
Changed lines of the file:
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@@
 	(footprint "VNLD5090-E:VNLD5090-E"
 		(layer "F.Cu")
-		(at 128.75 61.25 90)
+		(at 130.095 61.25 90)
 		(property "Reference" "U3"
 			(at -0.535 -3.637 90)
@@
 	)
 	(via
-		(at 133.75 61.5)
-		(size 0.8)
-		(drill 0.4)
-		(layers "F.Cu" "B.Cu")
-		(free yes)
-		(net 73)
-	)
-	(via
 		(at 183.25 119.3)
 		(size 0.8)
@@
 	)
 	(via
+		(at 127.5 61.25)
+		(size 0.8)
+		(drill 0.4)
+		(layers "F.Cu" "B.Cu")
+		(free yes)
+		(net 73)
+	)
+	(via
 		(at 121 127)
 		(size 0.8)
@@
 	)
 	(via
-		(at 129.75 67.25)
-		(size 0.8)
-		(drill 0.4)
-		(layers "F.Cu" "B.Cu")
-		(free yes)
-		(net 73)
-	)
-	(via
 		(at 143.5 122.25)
 		(size 0.8)
@@
 	)
 	(via
-		(at 131.75 55.75)
-		(size 0.8)
-		(drill 0.4)
-		(layers "F.Cu" "B.Cu")
-		(free yes)
-		(net 73)
-	)
-	(via
 		(at 211.5 48.25)
 		(size 0.8)
@@
 	)
 	(via
+		(at 131.25 61.25)
+		(size 0.8)
+		(drill 0.4)
+		(layers "F.Cu" "B.Cu")
+		(free yes)
+		(net 73)
+	)
+	(via
 		(at 200.5 56.75)
 		(size 0.8)
@@
 	)
 	(via
-		(at 210 77.25)
+		(at 132.5 61.25)
 		(size 0.8)
 		(drill 0.4)
@@
 	)
 	(via
-		(at 166 126)
+		(at 210 77.25)
 		(size 0.8)
 		(drill 0.4)
@@
 	)
 	(via
-		(at 130.75 56.75)
+		(at 166 126)
 		(size 0.8)
 		(drill 0.4)
@@
 	)
 	(via
+		(at 129.5 56.75)
+		(size 0.8)
+		(drill 0.4)
+		(layers "F.Cu" "B.Cu")
+		(free yes)
+		(net 73)
+	)
+	(via
 		(at 208.25 49.75)
 		(size 0.8)
@@
 	)
 	(via
-		(at 126.75 61)
+		(at 208.25 54.25)
 		(size 0.8)
 		(drill 0.4)
@@
 	)
 	(via
-		(at 208.25 54.25)
+		(at 138.75 97.75)
 		(size 0.8)
 		(drill 0.4)
@@
 	)
 	(via
-		(at 138.75 97.75)
+		(at 144.75 96.75)
 		(size 0.8)
 		(drill 0.4)
@@
 	)
 	(via
-		(at 144.75 96.75)
+		(at 162 69.25)
 		(size 0.8)
 		(drill 0.4)
@@
 	)
 	(via
-		(at 162 69.25)
+		(at 130.095 61.25)
 		(size 0.8)
 		(drill 0.4)
@@
 	)
 	(via
-		(at 130.75 61)
-		(size 0.8)
-		(drill 0.4)
-		(layers "F.Cu" "B.Cu")
-		(free yes)
-		(net 73)
-	)
-	(via
 		(at 204.5 48.25)
 		(size 0.8)
@@
 	)
 	(via
-		(at 128 56.75)
-		(size 0.8)
-		(drill 0.4)
-		(layers "F.Cu" "B.Cu")
-		(free yes)
-		(net 73)
-	)
-	(via
 		(at 150 65)
 		(size 0.8)
@@
 	)
 	(via
-		(at 129.25 61)
+		(at 133.25 58.75)
 		(size 0.8)
 		(drill 0.4)
@@
 	)
 	(via
-		(at 209 50.5)
+		(at 128.75 61.25)
 		(size 0.8)
 		(drill 0.4)
@@
 	)
 	(via
-		(at 119.75 112.75)
+		(at 209 50.5)
 		(size 0.8)
 		(drill 0.4)
@@
 	)
 	(via
-		(at 136.5 107.5)
+		(at 119.75 112.75)
 		(size 0.8)
 		(drill 0.4)
@@
 	)
 	(via
-		(at 132.25 58.75)
+		(at 136.5 107.5)
 		(size 0.8)
 		(drill 0.4)
@@
 		(net 73)
 	)
-	(via
-		(at 128 61)
-		(size 0.8)
-		(drill 0.4)
-		(layers "F.Cu" "B.Cu")
-		(free yes)
-		(net 73)
-	)
 	(segment
 		(start 123.725 79.615)
@@
 	)
 	(segment
-		(start 139.85 75.174999)
-		(end 129.385 64.709999)
-		(width 0.2)
+		(start 140.75 93.48)
+		(end 139.87 93.48)
+		(width 0.15)
 		(layer "F.Cu")
 		(net 76)
 	)
 	(segment
-		(start 140.75 93.48)
-		(end 139.87 93.48)
-		(width 0.15)
+		(start 146.275003 102.424998)
+		(end 139.85 95.999995)
+		(width 0.2)
 		(layer "F.Cu")
 		(net 76)
 	)
 	(segment
-		(start 139.85 93.5)
-		(end 139.85 75.174999)
+		(start 139.85 95.999995)
+		(end 139.85 93.5)
 		(width 0.2)
 		(layer "F.Cu")
@@
 	)
 	(segment
-		(start 146.275003 102.424998)
-		(end 139.85 95.999995)
+		(start 139.85 93.5)
+		(end 139.85 75.827208)
 		(width 0.2)
 		(layer "F.Cu")
@@
 	)
 	(segment
-		(start 139.85 95.999995)
-		(end 139.85 93.5)
+		(start 139.85 75.827208)
+		(end 130.73 66.707208)
 		(width 0.2)
 		(layer "F.Cu")
@@
 	)
 	(segment
-		(start 129.385 64.709999)
-		(end 129.385 63.725)
+		(start 130.73 66.707208)
+		(end 130.73 63.725)
 		(width 0.2)
 		(layer "F.Cu")
@@
 	)
 	(segment
-		(start 129.385 58.775)
-		(end 129.385 56.265)
+		(start 130.73 58.775)
+		(end 130.73 54.92)
 		(width 0.5)
 		(layer "F.Cu")
@@
 	)
 	(segment
-		(start 129.385 56.265)
+		(start 130.73 54.92)
 		(end 132.2 53.45)
 		(width 0.5)
@@
 	)
 	(segment
-		(start 126.845 50.595)
-		(end 125.2 48.95)
+		(start 127 50.75)
+		(end 127 55)
+		(width 0.5)
+		(layer "F.Cu")
+		(net 162)
+	)
+	(segment
+		(start 125.2 48.95)
+		(end 127 50.75)
 		(width 0.5)
 		(layer "F.Cu")
@@
 	)
 	(segment
-		(start 126.845 58.775)
-		(end 126.845 50.595)
+		(start 128.19 56.19)
+		(end 128.19 58.775)
+		(width 0.5)
+		(layer "F.Cu")
+		(net 162)
+	)
+	(segment
+		(start 127 55)
+		(end 128.19 56.19)
 		(width 0.5)
 		(layer "F.Cu")
@@
 	)
 	(segment
-		(start 139.5 96.449999)
-		(end 146.275 103.224999)
+		(start 128.19 63.725)
+		(end 128.19 64.051698)
 		(width 0.2)
 		(layer "F.Cu")
@@
 	)
 	(segment
-		(start 138.5 93.49)
-		(end 139.49 93.49)
-		(width 0.15)
+		(start 139.5 96.449999)
+		(end 146.275 103.224999)
+		(width 0.2)
 		(layer "F.Cu")
 		(net 163)
 	)
 	(segment
-		(start 129.465014 65.284987)
-		(end 139.5 75.319973)
+		(start 128.19 64.662182)
+		(end 139.5 75.972182)
 		(width 0.2)
 		(layer "F.Cu")
@@
 	)
 	(segment
-		(start 139.5 75.319973)
-		(end 139.5 93.5)
-		(width 0.2)
+		(start 138.5 93.49)
+		(end 139.49 93.49)
+		(width 0.15)
 		(layer "F.Cu")
 		(net 163)
 	)
 	(segment
-		(start 126.845 64.709999)
-		(end 127.419988 65.284987)
+		(start 139.5 75.972182)
+		(end 139.5 93.5)
 		(width 0.2)
 		(layer "F.Cu")
@@
 	)
 	(segment
-		(start 126.845 63.725)
-		(end 126.845 64.709999)
+		(start 128.19 63.725)
+		(end 128.19 64.662182)
 		(width 0.2)
 		(layer "F.Cu")
@@
 	)
 	(segment
-		(start 127.419988 65.284987)
-		(end 129.465014 65.284987)
-		(width 0.2)
-		(layer "F.Cu")
-		(net 163)
-	)
-	(segment
 		(start 139.49 93.49)
 		(end 139.5 93.5)
@@
 		(min_thickness 0.2)
 		(filled_areas_thickness no)
-		(fill yes
+		(fill
 			(thermal_gap 0.3)
 			(thermal_bridge_width 0.4)

Commit message: sync
Parts:
- added J5: Conn_02x02_Counter_Clockwise, Connector_Molex:Molex_Mini-Fit_Jr_5569-04A2_2x02_P4.20mm_Horizontal, F.Cu at (207.0, 124.5)
- moved C1 6.95 mm to (201.0, 114.8)
- moved C2 6.95 mm to (202.8, 118.0)
- moved U7 6.95 mm to (198.5, 118.0)
Routing:
- net /CAN2L: track 0.00 -> 21.2 mm
- net /CAN2H: track 0.00 -> 15.0 mm
- net +5VA: track 133.6 -> 124.2 mm
- net /EGT+: track 1.84 -> 10.6 mm
- net /EGT-: track 1.84 -> 8.43 mm
- net /CS3: track 48.8 -> 47.8 mm
- net /SCK3: track 48.2 -> 47.2 mm
- net /MISO3: track 48.8 -> 47.8 mm
- net GND: vias 258 -> 285
