File: AE101Corolla.kicad_pcb (KiCad board)
At the start: 4 copper layers, 100 x 100 mm, 44 parts, among them J1 175448-6, J2 6437288-2, J3 USB_C_Receptacle_USB2.0_14P, J4 Conn_02x03_Counter_Clockwise, J5 Conn_02x02_Counter_Clockwise, M1 Module-mega-mcu144-0.7, M2 Module-vr-discrete-0.5, M3 Module-vr-max9924-0.1, M4 Module-power_12and5V-0.3, M5 Module-knock-0.2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

Commit message: sync
Parts:
- added R11: 4.7k, Resistor_SMD:R_0402_1005Metric, B.Cu at (121.0, 73.8)
- added R12: 4.7k, Resistor_SMD:R_0402_1005Metric, B.Cu at (117.2, 73.8)
- added R13: 4.7k, Resistor_SMD:R_0402_1005Metric, B.Cu at (118.5, 73.8)
- added R14: 4.7k, Resistor_SMD:R_0402_1005Metric, B.Cu at (119.8, 73.8)
- moved J5 0.55 mm to (206.5, 124.4)
Connections:
- J5 pad 2: /CAN2L -> /CAN2H
- J5 pad 4: /CAN2H -> /CAN2L
Routing:
- net /INJ2_IN: track 58.0 -> 71.7 mm, vias 1 -> 3
- net /INJ3_IN: track 54.6 -> 63.7 mm, vias 1 -> 3
- net /CAN2L: track 21.2 -> 13.3 mm
- net /INJ4_IN: track 50.9 -> 57.4 mm, vias 1 -> 3
- net /CAN2H: track 15.0 -> 19.7 mm
- net /INJ1_IN: track 61.1 -> 62.5 mm
- net /OUT2: track 93.2 -> 92.2 mm
- net /IGN4: track 84.8 -> 84.0 mm
- net /IGN3: track 85.1 -> 84.6 mm
- net /IGN2: track 85.8 -> 85.3 mm
- net +12V_RAW: track 222.4 -> 221.9 mm
- net GND: vias 285 -> 292
