File: AE101Corolla.kicad_sch (KiCad schematic)
At the start: 16 parts, among them J1 175448-6, J2 175448-6, M1 Module-mega-mcu144-0.7, M2 Module-vr-discrete-0.5, M3 Module-vr-max9924-0.1, M4 Module-power_12and5V-0.3, M5 Module-knock-0.2

Commit message: sync
Parts:
- removed J1: 175448-6, 175448-6:1754486, symbol 175448-6:175448-6
- removed J2: 175448-6, symbol 175448-6:175448-6
- added J1: 175448-6, 175448-6:1754486, symbol 175448-6:175448-6_1
- added J2: 6437288-2, 6437288_2:TE_6437288-2, symbol 6437288-2:6437288-2
- added J3: USB_C_Receptacle_USB2.0_14P, Connector_USB:USB_C_Receptacle_GCT_USB4105-xx-A_16P_TopMnt_Horizontal, symbol Connector:USB_C_Receptacle_USB2.0_14P
- added M6: Module-can-0.1, can:can, symbol can:Module-can-0.1
- added R1, R2, R3, R4: 4.7k, Resistor_SMD:R_0402_1005Metric, symbol Device:R
- added R5, R6: 5.1k, Resistor_SMD:R_0402_1005Metric, symbol Device:R
- JP1: footprint (none) -> Jumper:SolderJumper-2_P1.3mm_Open_TrianglePad1.0x1.5mm
- M1: footprint megamcu144:mega-mcu144 -> mega-mcu144:mega-mcu144
- M3: footprint vrmax9924:vr-max9924 -> vr-max9924:vr-max9924
- M4: footprint power5_12:power_12and5V -> power_12and5V:power_12and5V
- M5: footprint hellen-one-knock-0.2:knock -> knock:knock
Connections:
- net +12V_PERM: now also M4.V1 (V12_PERM), J1.15 (BATT)
- net +12V_RAW: now also M4.V2 (IN_VIGN), M4.V3 (V12_RAW), J1.16 (+B1), J1.22 (+B)
- net +5V: now also M1.N31 (VCC), M4.E4 (V5)
- net +5VA: now also M1.E38 (V5A_SWITCHABLE), M5.E1 (V5A), M6.V1 (V5)
- net ACSTATUS: now also M1.S19 (IN_MAP3), J1.19 (AC1); no longer M1.S2 (IN_D3)
- net ACTEMP: now also J1.11 (ACT)
- net BOOSTSOLENOID_IN: now also R3.1
- net BOOSTSOLENOID_OUT: now also U3.8 (DRAIN1), J2.5; no longer U3.7 (SOURCE1)
- net CLT: now also J1.43 (THW)
- net ELECTRICLOAD: now also M1.S20 (IN_MAP2), J1.17 (ELS); no longer M1.S3 (IN_D2)
- net FUELRELAY_IN: now also R4.1
- net FUELRELAY_OUT: now also U3.6 (DRAIN2), J1.13 (FC); no longer U3.5 (SOURCE2)
- net GND: now also M4.S1 (GND), U3.5 (SOURCE2), U3.7 (SOURCE1), U4.5 (SOURCE2), U4.7 (SOURCE1), J1.1 (E01), J1.47 (E21), J1.6 (E02), J1.8 (E1), J1.MH1, J1.MH2, J1.MH3, J3.A1 (GND), J3.A12 (GND), J3.B1 (GND), J3.B12 (GND), J3.S1 (SHIELD), M6.E1 (GND), R1.2, R2.2, R3.2, R4.2, R5.1, R6.1
- net IACCLOSE_IN: now also R1.1
- net IACCLOSE_OUT: now also U4.8 (DRAIN1), J1.24 (RSC); no longer U4.7 (SOURCE1)
- net IACOPEN_IN: now also R2.1
- net IACOPEN_OUT: now also U4.6 (DRAIN2), J1.23 (RSO); no longer U4.5 (SOURCE2)
- net IAT: now also J1.44 (THA)
- net IDLSW: now also J1.51 (IDL)
- net INJ1_OUT: now also J1.2 (#10), J2.1
- net INJ2_OUT: now also J2.2
- net INJ3_OUT: now also J1.7 (#20), J2.3
- net INJ4_OUT: now also J2.4
- net KNOCK_RAW: now also J1.49 (KNK)
- net MAP: now also J1.45 (PIM)
- net NARROWO2_DOWNSTR: now also J1.42 (OX2)
- net NARROWO2_UPSTR: now also J1.41 (OX)
- net SPEED: now also J1.18 (SPD)
- net TPS: now also J1.53 (VTA)
- net VR+: now also J1.29 (NE+)
- net VR-: now also J1.37 (NE-)
- net VREF1: now reaches M5.W2 (VREF)
- net VREF1: now also M1.S35 (VREF1)
- net at M1.E1 (SPI2_SCK/CAN2_TX): now also M6.V5 (CAN_TX)
- net VR_THRESH: now reaches M1.E28 (OUT_PWM8)
- net VR_THRESH: now also M2.E1 (Thresh_IN)
- net at M1.E4 (SPI2_CS/CAN2_RX): now also M6.V6 (CAN_RX)
- net USB-: now reaches M1.N2 (USBM)
- net USB-: now also J3.A7 (D-), J3.B7 (D-)
- net VIGN: now reaches M1.N26 (IN_VIGN)
- net VIGN: now also M4.E3 (VIGN)
- net VBAT: now reaches M1.N27 (VBAT)
- net VBAT: now also M4.E1 (VBAT)
- net +3.3VA: now reaches M1.N28 (V33_SWITCHABLE)
- net +3.3VA: now also M6.V2 (CAN_VIO)
- net 5VP_ENABLE: now reaches M1.N29 (OUT_PWR_EN)
- net 5VP_ENABLE: now also M4.E5 (EN_5VP)
- net USB+: now reaches M1.N3 (USBP)
- net USB+: now also J3.A6 (D+), J3.B6 (D+)
- net at M1.N4 (VBUS): now also J3.A4 (VBUS), J3.A9 (VBUS), J3.B4 (VBUS), J3.B9 (VBUS)
- net AUX4: now reaches M1.S10 (IN_AUX4)
- net AUX4: now also J2.29
- net AUX3: now reaches M1.S11 (IN_AUX3)
- net AUX3: now also J2.28
- net AUX2: now reaches M1.S12 (IN_AUX2)
- net AUX2: now also J2.27
- net AUX1: now reaches M1.S13 (IN_AUX1)
- net AUX1: now also J2.26
- net RES2: now reaches M1.S14 (IN_RES2)
- net RES2: now also J2.19
- net RES1: now reaches M1.S17 (IN_RES1)
- net RES1: now also J2.18
- net RES3: now reaches M1.S18 (IN_RES3)
- net RES3: now also J2.20
- net D1: now reaches M1.S4 (IN_D1)
- net D1: now also J2.10
- net SENS4: now reaches M1.S6 (IN_SENS4)
- net SENS4: now also J2.24
- net SENS3: now reaches M1.S7 (IN_SENS3)
- net SENS3: now also J2.23
- net SENS2: now reaches M1.S8 (IN_SENS2)
- net SENS2: now also J2.22
- net SENS1: now reaches M1.S9 (IN_SENS1)
- net SENS1: now also J2.21
- net GNDA: now reaches M1.W1 (GNDA)
- net GNDA: now also J1.54 (E2), J2.14, J2.15
- net IGN2: now reaches M1.W10 (IGN2)
- net IGN2: now also J2.7
- net IGN1: now reaches M1.W11 (IGN1)
- net IGN1: now also J1.32 (IGT), J2.6
- net CAN1H: now reaches M1.W12 (CANH)
- net CAN1L: now reaches M1.W13 (CANL)
- net IGN4: now reaches M1.W8 (IGN4)
- net IGN4: now also J2.9
- net IGN3: now reaches M1.W9 (IGN3)
- net IGN3: now also J2.8
- net SYNC-: now reaches M2.W1 (VR-)
- net SYNC-: now also J1.36 (G-)
- net SYNC+: now reaches M2.W2 (VR+)
- net SYNC+: now also J1.28 (G1)
- net +5VP: now reaches M4.V4 (5VP)
- net +5VP: now also J1.52 (VC), J2.16, J2.17
- new net: J3.A5 (CC1), R6.2
- new net: J3.B5 (CC2), R5.2
- new net CAN2H: M6.S2 (CANH)
- new net CAN2L: M6.S1 (CANL)
- new net CHECKENGINE: J1.21 (W)
- new net D2: M1.S3 (IN_D2)
- new net D3: M1.S2 (IN_D3)
- new net NEUTRALSW: J1.9 (NSW)
- no-connect marks 8 -> 32
Other:
- note added: "ACT is ac condenser thermistor (ntc), input to ecu AC1 is 12v signal from ac computer to ecu, telling it ac has been switched on (for idle up) AC2 is signal from ecu to ac computer, telling it to engage clutch (allow ecu to disengage e.g full throttle)"
- note added: "THG is gas temp sensor for the egr passage EGR is solenoid to enable egr"
- note removed: "AC setup: ACT is condenser thermistor (ntc), input to ecu AC1 is 12v signal from ac computer to ecu, telling it ac has been switched on (for idle up) AC2 is signal from ecu to ac computer, telling it to engage clutch (allow ecu to disengage e.g full throttle)"
- moved on the sheet: D1, D2, D3, D4, M4

Commit message: sync
Parts:
- added D5, D6, D7, D8: B5819W, Diode_SMD:D_SOD-123, symbol Device:D_Schottky
- added R10, R7, R8, R9: 4.7k, Resistor_SMD:R_0402_1005Metric, symbol Device:R
- added U5, U6: ~, VNLD5090-E:VNLD5090-E, symbol VNLD5090-E:VNLD5090-E
Connections:
- net CHECKENGINE is gone; now on net CHECKENGINE_OUT: J1.21 (W)
- net +12V_RAW: now also D5.1 (K), D6.1 (K), D7.1 (K), D8.1 (K)
- net +5V: no longer JP1.2 (B)
- net +5VA: now also JP1.2 (B)
- net AUX1: no longer J2.26
- net AUX2: no longer J2.27
- net AUX3: no longer J2.28
- net AUX4: no longer J2.29
- net D1: no longer J2.10
- net FUELRELAY_IN: now also M1.E19 (OUT_INJ1); no longer M1.E31 (OUT_INJ5)
- net GND: now also U1.6 (DRAIN2), U1.8 (DRAIN1), R10.2, R7.2, R8.2, R9.2, U5.5 (SOURCE2), U5.7 (SOURCE1), U6.5 (SOURCE2), U6.7 (SOURCE1); no longer J1.47 (E21)
- net GNDA: now also J1.47 (E21)
- net IACOPEN_IN: now also M1.E26 (OUT_PWM6); no longer M1.E17 (OUT_PWM2)
- net IGN1: no longer J2.6
- net IGN2: no longer J2.7
- net IGN3: no longer J2.8
- net IGN4: no longer J2.9
- net INJ1_IN: now also M1.E34 (OUT_INJ8); no longer M1.E19 (OUT_INJ1)
- net INJ1_OUT: now also J2.34; no longer J2.1
- net INJ2_IN: now also M1.E33 (OUT_INJ7); no longer M1.E18 (OUT_INJ2)
- net INJ2_OUT: now also J2.33; no longer J2.2
- net INJ3_IN: now also M1.E32 (OUT_INJ6); no longer M1.E29 (OUT_INJ3)
- net INJ3_OUT: now also J2.32; no longer J2.3
- net INJ4_IN: now also M1.E31 (OUT_INJ5); no longer M1.E30 (OUT_INJ4)
- net INJ4_OUT: now also J2.31; no longer J2.4
- net RES1: no longer J2.18
- net RES2: no longer J2.19
- net RES3: no longer J2.20
- net SENS1: no longer J2.21
- net SENS2: no longer J2.22
- net SENS3: no longer J2.23
- net SENS4: no longer J2.24
- net LS3_IN: now reaches M1.E14 (OUT_PWM5)
- net LS3_IN: now also R8.1, U6.1 (IN1)
- net LS2_IN: now reaches M1.E15 (OUT_PWM4)
- net LS2_IN: now also R9.1, U5.3 (IN2)
- net LS1_OUT: now reaches J2.30
- net LS1_OUT: now also D7.2 (A), U5.8 (DRAIN1)
- net BOOSTSOLENOID_IN renamed CHECKENGINE_IN
- net CHECKENGINE_IN: now also M1.E18 (OUT_INJ2); no longer M1.E16 (OUT_PWM3)
- net BOOSTSOLENOID_OUT renamed CHECKENGINE_OUT
- net CHECKENGINE_OUT: no longer J2.5
- new net LS1_IN: M1.E16 (OUT_PWM3), R7.1, U5.1 (IN1)
- new net LS2_OUT: D5.2 (A), J2.29, U5.6 (DRAIN2)
- new net LS3_OUT: D8.2 (A), J2.28, U6.8 (DRAIN1)
- new net LS4_IN: M1.E17 (OUT_PWM2), R10.1, U6.3 (IN2)
- new net LS4_OUT: D6.2 (A), J2.27, U6.6 (DRAIN2)
- no-connect marks 32 -> 36
Other:
- moved on the sheet: J1

Commit message: sync
Parts:
- added M7: Module-wbo-0.5, wbo:wbo, symbol wbo:Module-wbo-0.5
- J2: footprint 6437288_2:TE_6437288-2 -> superseal_34:TE_6437288-2
- M1: footprint mega-mcu144:mega-mcu144 -> megamcu144:mega-mcu144
- M3: footprint vr-max9924:vr-max9924 -> vrmax9924:vr-max9924
- M4: footprint power_12and5V:power_12and5V -> power5_12:power_12and5V
Connections:
- net +3.3VA: now also M7.W2 (CAN_VIO)
- net +5VA: now also M1.N30 (V5A_SWITCHABLE), M1.W2 (V5A_SWITCHABLE)
- net ACTEMP: now also M1.S27 (IN_AT1)
- net AUX1: now also J2.10
- net AUX2: now also J2.11
- net AUX3: now also J2.12
- net AUX4: now also J2.13
- net CAN1H: now also M7.W4 (CANH)
- net CAN1L: now also M7.W3 (CANL)
- net D1: now also J2.9
- net D2: now also J2.21
- net D3: now also J2.26
- net GND: now also U1.5 (SOURCE2), U1.7 (SOURCE1), U2.5 (SOURCE2), U2.7 (SOURCE1); no longer U1.6 (DRAIN2), U1.8 (DRAIN1), U2.6 (DRAIN2), U2.8 (DRAIN1)
- net GNDA: now also M1.E39 (GNDA)
- net IGN1: now also J2.1
- net IGN2: now also J2.2
- net IGN3: now also J2.3
- net IGN4: now also J2.4
- net INJ1_IN: now also M1.E32 (OUT_INJ6); no longer M1.E34 (OUT_INJ8)
- net INJ1_OUT: now also J2.30, U1.8 (DRAIN1); no longer J1.2 (#10), J2.34, U1.7 (SOURCE1)
- net INJ2_IN: now also M1.E31 (OUT_INJ5); no longer M1.E33 (OUT_INJ7)
- net INJ2_OUT: now also J2.29, U1.6 (DRAIN2); no longer J2.33, U1.5 (SOURCE2)
- net INJ3_IN: now also M1.E30 (OUT_INJ4); no longer M1.E32 (OUT_INJ6)
- net INJ3_OUT: now also J2.28, U2.8 (DRAIN1); no longer J1.7 (#20), J2.32, U2.7 (SOURCE1)
- net INJ4_IN: now also M1.E29 (OUT_INJ3); no longer M1.E31 (OUT_INJ5)
- net INJ4_OUT: now also J2.27, U2.6 (DRAIN2); no longer J2.31, U2.5 (SOURCE2)
- net LS1_IN: now also M1.E17 (OUT_PWM2); no longer M1.E16 (OUT_PWM3)
- net LS1_OUT: now also J2.34; no longer J2.30
- net LS2_IN: now also M1.E16 (OUT_PWM3); no longer M1.E15 (OUT_PWM4)
- net LS2_OUT: now also J2.33; no longer J2.29
- net LS3_IN: now also M1.E15 (OUT_PWM4); no longer M1.E14 (OUT_PWM5)
- net LS3_OUT: now also J2.32; no longer J2.28
- net LS4_IN: now also M1.E14 (OUT_PWM5); no longer M1.E17 (OUT_PWM2)
- net LS4_OUT: now also J2.31; no longer J2.27
- net RES1: now also J2.18
- net RES2: now also J2.20
- net RES3: now also J2.19
- net SENS1: now also J2.5
- net SENS2: now also J2.6
- net SENS3: now also J2.7
- net SENS4: now also J2.8
- net OUT4: now reaches M1.W4 (IGN8)
- net OUT4: now also J2.25
- net OUT3: now reaches M1.W5 (IGN7)
- net OUT3: now also J2.24
- net OUT2: now reaches M1.W6 (IGN6)
- net OUT2: now also J2.23
- net OUT1: now reaches M1.W7 (IGN5)
- net OUT1: now also J2.22
- no-connect marks 36 -> 38

Commit message: sync
Parts:
- D1, D2, D3, D4, D5, D6, D7, D8: LCSC (none) -> C8598
- R1, R10, R2, R3, R4, R7, R8, R9: LCSC (none) -> C4033814
- R5, R6: LCSC (none) -> C105872
- U1, U2, U3, U4, U5, U6: LCSC (none) -> C222209

Commit message: sync
Parts:
- added J4: Conn_02x03_Counter_Clockwise, Connector_Molex:Molex_Mini-Fit_Jr_5569-06A2_2x03_P4.20mm_Horizontal, symbol Connector_Generic:Conn_02x03_Counter_Clockwise
Connections:
- net +12V_RAW: now also J4.2 (Pin_2)
- net +3.3VA: no longer M7.W2 (CAN_VIO)
- net +5VA: now also M7.W1 (V5_IN)
- net GND: now also M7.E6 (LSU_H-), M7.G (GND)
- net at M7.E1 (LSU_Un): now also J4.6 (Pin_6)
- net at M7.E2 (LSU_Vm): now also J4.4 (Pin_4)
- net at M7.E3 (LSU_Ip): now also J4.3 (Pin_3)
- net at M7.E4 (LSU_Rtrim): now also J4.1 (Pin_1)
- net at M7.E5 (LSU_H+): now also J4.5 (Pin_5)
- net at M7.J1 (SEL1): now also M7.J_GND1 (PULL_DOWN1)
- no-connect marks 38 -> 48

Commit message: sync
Parts:
- added C1: 100n, Capacitor_SMD:C_0402_1005Metric, symbol Device:C
- added C2: 10n, Capacitor_SMD:C_0402_1005Metric, symbol Device:C
- added U7: MAX31855KASA, Package_SO:SOIC-8_3.9x4.9mm_P1.27mm, symbol Sensor_Temperature:MAX31855KASA
- R1, R10, R2, R3, R4, R7, R8, R9: LCSC C4033814 -> C25900
- R5, R6: LCSC C105872 -> C25900
Connections:
- net +5VA: now also C1.1, U7.4 (V_{CC}); no longer M1.E38 (V5A_SWITCHABLE)
- net GND: now also C1.2, U7.1 (GND)
- net GNDA: no longer M1.W1 (GNDA)
- net VREF1: now also M1.S5 (VREF2); no longer M1.S35 (VREF1)
- net CS3: now reaches M1.N10 (SPI3_CS)
- net CS3: now also U7.6 (~{CS})
- net SCK3: now reaches M1.N11 (SPI3_SCK)
- net SCK3: now also U7.5 (SCK)
- net MISO3: now reaches M1.N12 (SPI3_MISO)
- net MISO3: now also U7.7 (SO)
- new net EGT+: C2.2, U7.3 (T+)
- new net EGT-: C2.1, U7.2 (T-)
- no-connect marks 48 -> 52

Commit message: sync
Parts:
- R5, R6: LCSC C25900 -> C144745
Changed lines of the file:
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@@
 			)
 		)
-		(property "LCSC" "C25900"
+		(property "LCSC" "C144745"
 			(at 250.19 130.81 0)
 			(effects
@@
 			)
 		)
-		(property "LCSC" "C25900"
+		(property "LCSC" "C144745"
 			(at 259.08 130.81 0)
 			(effects

Commit message: sync
Parts:
- added J5: Conn_02x02_Counter_Clockwise, Connector_Molex:Molex_Mini-Fit_Jr_5569-04A2_2x02_P4.20mm_Horizontal, symbol Connector_Generic:Conn_02x02_Counter_Clockwise
Connections:
- net CAN2H: now also J5.4 (Pin_4)
- net CAN2L: now also J5.2 (Pin_2)
- net EGT+: now also J5.1 (Pin_1)
- net EGT-: now also J5.3 (Pin_3)
Changed lines of the file:
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@@
+		)
+	)
+	(label "CAN2H"
+		(at 284.48 218.44 270)
+		(effects
+			(font
+				(size 1.27 1.27)
+			)
+			(justify right bottom)
 		)
 	)
@@
 		)
 	)
+	(label "CAN2L"
+		(at 281.94 205.74 90)
+		(effects
+			(font
+				(size 1.27 1.27)
+			)
+			(justify left bottom)
+		)
+	)
 	(label "LS3_IN"
 		(at 91.44 171.45 0)
@@
 		)
 	)
-	(label "CAN2H"
-		(at 88.9 234.95 0)
-		(effects
-			(font
-				(size 1.27 1.27)
-			)
-			(justify left bottom)
-		)
-	)
 	(label "VR-"
 		(at 63.5 245.11 0)
@@
 		)
 	)
-	(label "CAN2L"
-		(at 88.9 232.41 0)
-		(effects
-			(font
-				(size 1.27 1.27)
-			)
-			(justify left bottom)
-		)
-	)
 	(label "MISO3"
 		(at 229.87 41.91 0)
@@
 		)
 	)
+	(label "EGT-"
+		(at 281.94 218.44 270)
+		(effects
+			(font
+				(size 1.27 1.27)
+			)
+			(justify right bottom)
+		)
+	)
 	(label "SCK3"
 		(at 280.67 187.96 0)
@@
 			)
 			(justify right bottom)
+		)
+	)
+	(label "EGT+"
+		(at 284.48 205.74 90)
+		(effects
+			(font
+				(size 1.27 1.27)
+			)
+			(justify left bottom)
 		)
 	)
@@
 					(unit 1)
 				)
+			)
+		)
+	)
+	(symbol
+		(lib_id "Connector_Generic:Conn_02x02_Counter_Clockwise")
+		(at 284.48 210.82 270)
+		(unit 1)
+		(exclude_from_sim no)
+		(in_bom yes)
+		(on_board yes)
+		(dnp no)
+		(fields_autoplaced yes)
+		(property "Reference" "J5"
+			(at 287.02 212.0899 90)
+			(effects
+				(font
+					(size 1.27 1.27)
+				)
+				(justify left)
+			)
+		)
+		(property "Value" "Conn_02x02_Counter_Clockwise"
+			(at 288.29 212.09 0)
+			(effects
+				(font
+					(size 1.27 1.27)
+				)
+				(hide yes)
+			)
+		)
+		(property "Footprint" "Connector_Molex:Molex_Mini-Fit_Jr_5569-04A2_2x02_P4.20mm_Horizontal"
+			(at 284.48 210.82 0)
+			(effects
+				(font
+					(size 1.27 1.27)
+				)
+				(hide yes)
+			)
+		)
+		(property "Datasheet" "~"
+			(at 284.48 210.82 0)
+			(effects
+				(font
+					(size 1.27 1.27)
+				)
+				(hide yes)
+			)
+		)
+		(property "Description" "Generic connector, double row, 02x02, counter clockwise pin numbering scheme (similar to DIP package numbering), script generated (kicad-library-utils/schlib/autogen/connector/)"
+			(at 284.48 210.82 0)
+			(effects
+				(font
+					(size 1.27 1.27)
+				)
+				(hide yes)
+			)
+		)
+		(pin "3"
+		)
+		(pin "1"
+		)
+		(pin "2"
+		)
+		(pin "4"
+		)
+		(instances
+			(project ""
+				(path "/70a65c1d-c703-4ce7-9653-99ac3171341d"
+					(reference "J5")
+					(unit 1)
+				)
