File: AE101Corolla.kicad_sch (KiCad schematic)
At the start: 40 parts, among them J1 175448-6, J2 6437288-2, J3 USB_C_Receptacle_USB2.0_14P, J4 Conn_02x03_Counter_Clockwise, J5 Conn_02x02_Counter_Clockwise, M1 Module-mega-mcu144-0.7, M2 Module-vr-discrete-0.5, M3 Module-vr-max9924-0.1, M4 Module-power_12and5V-0.3, M5 Module-knock-0.2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

Commit message: sync
Parts:
- added R11, R12, R13, R14: 4.7k, Resistor_SMD:R_0402_1005Metric, symbol Device:R
Connections:
- net CAN2H: now also J5.2 (Pin_2); no longer J5.4 (Pin_4)
- net CAN2L: now also J5.4 (Pin_4); no longer J5.2 (Pin_2)
- net GND: now also R11.2, R12.2, R13.2, R14.2
- net INJ1_IN: now also R11.1
- net INJ2_IN: now also R12.1
- net INJ3_IN: now also R13.1
- net INJ4_IN: now also R14.1
Other:
- moved on the sheet: C1, C2, D1, D2, D3, D4, D5, D6, D7, D8, J1, J2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
